Commit message: Add dataset generation, VR teleop, Isaac integration, and various improvements

File: src/ur5_robotiq_description/urdf/robotiq_2f85_original.urdf.xacro (robot description, xacro)
@@ -74,6 +74,6 @@
         <mass value="0.018491" />
         <origin xyz="0.0 0.0 0.0" />
-        <inertia ixx="0.000009" ixy="0.000000" ixz="0.000000"
-                 iyx="0.000000" iyy="0.000009" iyz="0.000000"
+        <inertia ixx="0.000009" ixy="-0.000001" ixz="0.000000"
+                 iyx="-0.000001" iyy="0.000001" iyz="0.000000"
                  izx="0.000000" izy="0.000000" izz="0.000010" />
       </inertial>
@@ -101,6 +101,6 @@
         <mass value="0.018491" />
         <origin xyz="0.0 0.0 0.0" />
-        <inertia ixx="0.000009" ixy="0.000000" ixz="0.000000"
-                 iyx="0.000000" iyy="0.000009" iyz="0.000000"
+        <inertia ixx="0.000009" ixy="-0.000001" ixz="0.000000"
+                 iyx="-0.000001" iyy="0.000001" iyz="0.000000"
                  izx="0.000000" izy="0.000000" izz="0.000010" />
       </inertial>
